Commit message: Corrected file references in sentry.xacro

File: urdf/sentry.xacro (robot description, xacro)
@@ -13,5 +13,5 @@
     <origin rpy="0 0 0" xyz="0 0 0"/>
     <geometry>
-      <mesh filename="package://sim_sentry/model/sentry/meshes/CAD/base_link.obj" scale="0.001 0.001 0.001"/>
+      <mesh filename="package://sim_sentry/meshes/base_link.stl" scale="0.001 0.001 0.001"/>
     </geometry>
     <material name="silver"/>
@@ -20,5 +20,5 @@
     <origin rpy="0 0 0" xyz="0 0 0"/>
     <geometry>
-      <mesh filename="package://sim_sentry/model/sentry/meshes/CAD/base_link.obj" scale="0.001 0.001 0.001"/>
+      <mesh filename="package://sim_sentry/meshes/base_link.stl" scale="0.001 0.001 0.001"/>
     </geometry>
   </collision>
@@ -34,5 +34,5 @@
     <origin rpy="0 0 0" xyz="0 0 0"/>
     <geometry>
-      <mesh filename="package://sim_sentry/model/sentry/meshes/CAD/wheel.obj" scale="0.001 0.001 0.001"/>
+      <mesh filename="package://sim_sentry/meshes/wheel.stl" scale="0.001 0.001 0.001"/>
     </geometry>
     <material name="silver"/>
@@ -41,5 +41,5 @@
     <origin rpy="0 0 0" xyz="0 0 0"/>
     <geometry>
-      <mesh filename="package://sim_sentry/model/sentry/meshes/CAD/wheel.obj" scale="0.001 0.001 0.001"/>
+      <mesh filename="package://sim_sentry/meshes/wheel.stl" scale="0.001 0.001 0.001"/>
     </geometry>
   </collision>
@@ -55,5 +55,5 @@
     <origin rpy="0 0 0" xyz="0 0 0"/>
     <geometry>
-      <mesh filename="package://sim_sentry/model/sentry/meshes/CAD/wheel.obj" scale="0.001 0.001 0.001"/>
+      <mesh filename="package://sim_sentry/meshes/wheel.stl" scale="0.001 0.001 0.001"/>
     </geometry>
     <material name="silver"/>
@@ -62,5 +62,5 @@
     <origin rpy="0 0 0" xyz="0 0 0"/>
     <geometry>
-      <mesh filename="package://sim_sentry/model/sentry/meshes/CAD/wheel.obj" scale="0.001 0.001 0.001"/>
+      <mesh filename="package://sim_sentry/meshes/wheel.stl" scale="0.001 0.001 0.001"/>
     </geometry>
   </collision>

Commit message: First working model

File: urdf/sentry.xacro (robot description, xacro)
@@ -67,16 +67,16 @@
 </link>
 <joint name="left_wheel_joint" type="continuous">
-  <origin rpy="0 0 1.5708" xyz="-0.18650 -0.20000099435655025 0.150"/>
+  <origin rpy="0 0 0" xyz="-0.18650 0 0.07260"/>
   <parent link="base_link"/>
   <child link="left_wheel"/>
-  <axis xyz="0.0 1.0 0.0"/>
+  <axis xyz="1.0 0.0 0.0"/>
   <limit effort="10000" velocity="1000"/>
   <joint_properties damping="1.0" friction="1.0"/>
 </joint>
 <joint name="right_wheel_joint" type="continuous">
-  <origin rpy="0 0 1.5708" xyz="0.18650 -0.20000099435655025 0.150"/>
+  <origin rpy="0 0 0" xyz="0.18650 0 0.07260"/>
   <parent link="base_link"/>
   <child link="right_wheel"/>
-  <axis xyz="0.0 1.0 0.0"/>
+  <axis xyz="1.0 0.0 0.0"/>
   <limit effort="10000" velocity="1000"/>
   <joint_properties damping="1.0" friction="1.0"/>

Commit message: Changed mesh uri

File: urdf/sentry.xacro (robot description, xacro)
@@ -16,5 +16,5 @@
     <origin rpy="0 0 0" xyz="0 0 0"/>
     <geometry>
-      <mesh filename="package://sim_sentry/meshes/base_link.stl" scale="0.001 0.001 0.001"/>
+      <mesh filename="package://sentry_description/meshes/base_link.stl" scale="0.001 0.001 0.001"/>
     </geometry>
     <material name="silver"/>
@@ -23,5 +23,5 @@
     <origin rpy="0 0 0" xyz="0 0 0"/>
     <geometry>
-      <mesh filename="package://sim_sentry/meshes/base_link.stl" scale="0.001 0.001 0.001"/>
+      <mesh filename="package://sentry_description/meshes/base_link.stl" scale="0.001 0.001 0.001"/>
     </geometry>
   </collision>
@@ -39,5 +39,5 @@
     <origin rpy="0 0 0" xyz="0 0 0"/>
     <geometry>
-      <mesh filename="package://sim_sentry/meshes/wheel.stl" scale="0.001 0.001 0.001"/>
+      <mesh filename="package://sentry_description/meshes/wheel.stl" scale="0.001 0.001 0.001"/>
     </geometry>
     <material name="silver"/>
@@ -46,5 +46,5 @@
     <origin rpy="0 0 0" xyz="0 0 0"/>
     <geometry>
-      <mesh filename="package://sim_sentry/meshes/wheel.stl" scale="0.001 0.001 0.001"/>
+      <mesh filename="package://sentry_description/meshes/wheel.stl" scale="0.001 0.001 0.001"/>
     </geometry>
   </collision>
@@ -60,5 +60,5 @@
     <origin rpy="0 0 0" xyz="0 0 0"/>
     <geometry>
-      <mesh filename="package://sim_sentry/meshes/wheel.stl" scale="0.001 0.001 0.001"/>
+      <mesh filename="package://sentry_description/meshes/wheel.stl" scale="0.001 0.001 0.001"/>
     </geometry>
     <material name="silver"/>
@@ -67,5 +67,5 @@
     <origin rpy="0 0 0" xyz="0 0 0"/>
     <geometry>
-      <mesh filename="package://sim_sentry/meshes/wheel.stl" scale="0.001 0.001 0.001"/>
+      <mesh filename="package://sentry_description/meshes/wheel.stl" scale="0.001 0.001 0.001"/>
     </geometry>
   </collision>
